File: tillmann-preamp.kicad_sch (KiCad schematic)
At the start: 12 parts, among them J1 AudioJack3_Switch, J2 Input Signal, J3 AudioJack3_Switch, J4 Output Signal, J5 Barrel_Jack, Q1 Q_NJFET_DGS

Commit message: Update PCB for milling v1.0
Parts:
- added J6: 9V, Connector_PinHeader_2.54mm:PinHeader_1x02_P2.54mm_Vertical, symbol Connector_Generic:Conn_01x02
- C1, C2: footprint Capacitor_THT:CP_Radial_D8.0mm_P3.50mm -> Capacitor_THT:CP_Radial_D5.0mm_P2.50mm
- Q1: Comments (none) -> J110 was used in this design, BFW13 and 2N3438 are alternat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
Connections:
- net +9V: now also J6.2 (Pin_2)
- net GND: now also J6.1 (Pin_1)
Other:
- company: (none) -> Besmer Labs
- title: (none) -> Tillman Preamp
Changed lines of the file:
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@@
 (kicad_sch (version 20211123) (generator eeschema)
   (paper "A4")
+  (title_block
+    (title "Tillman Preamp")
+    (date "2023-02-06")
+    (rev "1.0")
+    (company "Besmer Labs")
+  )
   (junction (at 173.228 80.772) (diameter 0) (color 0 0 0 0)
   )
@@
     (stroke (width 0) (type default) (color 0 0 0 0))
   )
+  (wire (pts (xy 152.654 53.594) (xy 162.56 53.594))
+    (stroke (width 0) (type default) (color 0 0 0 0))
+  )
   (wire (pts (xy 161.544 75.692) (xy 161.544 80.772))
     (stroke (width 0) (type default) (color 0 0 0 0))
@@
     (stroke (width 0) (type default) (color 0 0 0 0))
   )
+  (wire (pts (xy 162.56 47.752) (xy 159.766 47.752))
+    (stroke (width 0) (type default) (color 0 0 0 0))
+  )
   (wire (pts (xy 111.506 87.376) (xy 113.538 87.376))
     (stroke (width 0) (type default) (color 0 0 0 0))
@@
     (stroke (width 0) (type default) (color 0 0 0 0))
   )
+  (wire (pts (xy 159.766 47.752) (xy 159.766 45.974))
+    (stroke (width 0) (type default) (color 0 0 0 0))
+  )
   (wire (pts (xy 118.11 87.376) (xy 118.11 88.392))
     (stroke (width 0) (type default) (color 0 0 0 0))
@@
     (stroke (width 0) (type default) (color 0 0 0 0))
   )
-  (wire (pts (xy 152.654 53.594) (xy 147.066 53.594))
+  (wire (pts (xy 147.066 53.594) (xy 152.654 53.594))
+    (stroke (width 0) (type default) (color 0 0 0 0))
+  )
+  (wire (pts (xy 162.56 53.594) (xy 162.56 50.292))
     (stroke (width 0) (type default) (color 0 0 0 0))
   )
@@
     (stroke (width 0) (type default) (color 0 0 0 0))
   )
-  (wire (pts (xy 152.654 45.974) (xy 147.066 45.974))
+  (wire (pts (xy 147.066 45.974) (xy 152.654 45.974))
     (stroke (width 0) (type default) (color 0 0 0 0))
   )
@@
   )
   (wire (pts (xy 161.544 80.772) (xy 155.702 80.772))
+    (stroke (width 0) (type default) (color 0 0 0 0))
+  )
+  (wire (pts (xy 159.766 45.974) (xy 152.654 45.974))
     (stroke (width 0) (type default) (color 0 0 0 0))
   )
@@
     )
     (property "Datasheet" "~" (id 3) (at 130.302 87.376 0)
+      (effects (font (size 1.27 1.27)) hide)
+    )
+    (property "Comments" "J110 was used in this design, BFW13 and 2N3438 are alternatives too" (id 4) (at 130.302 87.376 0)
       (effects (font (size 1.27 1.27)) hide)
     )
@@
       (effects (font (size 1.27 1.27)) (justify left))
     )
-    (property "Footprint" "Capacitor_THT:CP_Radial_D8.0mm_P3.50mm" (id 2) (at 153.6192 53.594 0)
+    (property "Footprint" "Capacitor_THT:CP_Radial_D5.0mm_P2.50mm" (id 2) (at 153.6192 53.594 0)
       (effects (font (size 1.27 1.27)) hide)
     )
@@
     (pin "2")
   )
+  (symbol (lib_id "Connector_Generic:Conn_01x02") (at 167.64 50.292 0) (mirror x) (unit 1)
+    (in_bom yes) (on_board yes) (fields_autoplaced)
+    (property "Reference" "J6" (id 0) (at 167.64 41.656 0))
+    (property "Value" "9V" (id 1) (at 167.64 44.196 0))
+    (property "Footprint" "Connector_PinHeader_2.54mm:PinHeader_1x02_P2.54mm_Vertical" (id 2) (at 167.64 50.292 0)
+      (effects (font (size 1.27 1.27)) hide)
+    )
+    (property "Datasheet" "~" (id 3) (at 167.64 50.292 0)
+      (effects (font (size 1.27 1.27)) hide)
+    )
+    (pin "1")
+    (pin "2")
+  )
   (symbol (lib_id "Device:C_Polarized") (at 151.892 80.772 90) (unit 1)
     (in_bom yes) (on_board yes) (fields_autoplaced)
     (property "Reference" "C1" (id 0) (at 151.003 73.66 90))
     (property "Value" "4.7u" (id 1) (at 151.003 76.2 90))
-    (property "Footprint" "Capacitor_THT:CP_Radial_D8.0mm_P3.50mm" (id 2) (at 155.702 79.8068 0)
+    (property "Footprint" "Capacitor_THT:CP_Radial_D5.0mm_P2.50mm" (id 2) (at 155.702 79.8068 0)
       (effects (font (size 1.27 1.27)) hide)
     )
@@
     )
     (path "/d7a28c4c-9204-4215-8b0c-d275e4a21d05"
-      (reference "C1") (unit 1) (value "4.7u") (footprint "Capacitor_THT:CP_Radial_D8.0mm_P3.50mm")
+      (reference "C1") (unit 1) (value "4.7u") (footprint "Capacitor_THT:CP_Radial_D5.0mm_P2.50mm")
     )
     (path "/a2b042eb-65d4-49f6-8432-95c8b36b1907"
-      (reference "C2") (unit 1) (value "10u") (footprint "Capacitor_THT:CP_Radial_D8.0mm_P3.50mm")
+      (reference "C2") (unit 1) (value "10u") (footprint "Capacitor_THT:CP_Radial_D5.0mm_P2.50mm")
     )
     (path "/8e531742-efd7-4dcf-9a8c-90495eb4f8ed"
@@
       (reference "J5") (unit 1) (value "Barrel_Jack") (footprint "Connector_BarrelJack:BarrelJack_CUI_PJ-063AH_Horizontal")
     )
+    (path "/d32bd163-7f85-4111-a0ac-d1e935f84d9c"
+      (reference "J6") (unit 1) (value "9V") (footprint "Connector_PinHeader_2.54mm:PinHeader_1x02_P2.54mm_Vertical")
+    )
     (path "/88ce6874-c519-4585-8adb-dac376e88ba7"
